File: W5500-hat.kicad_pcb (KiCad board)
At the start: 2 copper layers, 22.9 x 55.9 mm, 28 parts, among them J1 Conn, J2 Conn, J3 RB1-125BAG1A, J4 Conn, J5 Conn, J8 RJ45_Amphenol_RJMG1BD3B8K1ANR, SW2 SW_Push, U5 W5500, U6 74AHC1G125, Y1 24MHz

Commit message: Tracks almost finished
Parts:
- added C10: 100nF, Capacitor_SMD:C_0402_1005Metric, F.Cu at (141.5, 102.1)
- added C11: 100nF, Capacitor_SMD:C_0402_1005Metric, F.Cu at (141.5, 103.1)
- added C12: 1uF, Capacitor_SMD:C_0603_1608Metric, F.Cu at (141.2, 104.3)
- added C4: 10uF, Capacitor_SMD:C_0603_1608Metric, F.Cu at (145.7, 90.0)
- added C5: 100nF, Capacitor_SMD:C_0402_1005Metric, F.Cu at (142.6, 90.0)
- added C6: 1uF, Capacitor_SMD:C_0603_1608Metric, F.Cu at (131.8, 82.1)
- added C7: 100nF, Capacitor_SMD:C_0402_1005Metric, F.Cu at (131.5, 83.3)
- added JP1: JMP, Jumper:SolderJumper-2_P1.3mm_Open_RoundedPad1.0x1.5mm, B.Cu at (133.5, 103.7)
- added JP2: JMP, Jumper:SolderJumper-2_P1.3mm_Open_RoundedPad1.0x1.5mm, B.Cu at (131.3, 103.7)
- added JP3: JMP, Jumper:SolderJumper-2_P1.3mm_Open_RoundedPad1.0x1.5mm, B.Cu at (135.8, 103.7)
- added R4: 10K, Resistor_SMD:R_0402_1005Metric, F.Cu at (131.0, 100.9)
- added R5: 10K, Resistor_SMD:R_0402_1005Metric, F.Cu at (130.0, 100.9)
- added R6: 10K, Resistor_SMD:R_0402_1005Metric, F.Cu at (132.0, 100.9)
- added R7: 49.9, Resistor_SMD:R_0402_1005Metric, F.Cu at (140.5, 80.8)
- added R8: 17.4K, Resistor_SMD:R_0402_1005Metric, F.Cu at (138.2, 100.7)
- C9: value 1uF -> 100nF; footprint Capacitor_SMD:C_0603_1608Metric -> Capacitor_SMD:C_0402_1005Metric
- moved FB2 17.6 mm to (142.6, 87.4), turned to -90 degrees
- moved C9 6.56 mm to (141.5, 101.1), turned to 180 degrees
- moved FB1 6.04 mm to (133.7, 106.8), turned to -90 degrees
- moved C18 4.58 mm to (136.0, 112.0), turned to -90 degrees
- moved C8 1.51 mm to (141.5, 100.1), turned to 180 degrees
- moved SW2 0.43 mm to (145.5, 83.3)
- moved C3 0.13 mm to (131.8, 89.1)
- moved U6 0.12 mm to (132.5, 86.9)
Connections:
- C8 pad 1: +1V2 -> AVDD
- C8 pad 2: GND -> AGND
- C9 pad 1: +1V2 -> AVDD
- C9 pad 2: GND -> AGND
- SW2 pad 1: unconnected-(SW2-Pad1) -> GND
- SW2 pad 2: unconnected-(SW2-Pad2) -> /~{RST}
- U5 pad 10: unconnected-(U5-EXRES1-Pad10) -> Net-(U5-EXRES1)
- U5 pad 11: Net-(U5-AVDD-Pad11) -> AVDD
- U5 pad 14: GND -> AGND
- U5 pad 15: Net-(U5-AVDD-Pad11) -> AVDD
- U5 pad 16: GND -> AGND
- U5 pad 17: Net-(U5-AVDD-Pad11) -> AVDD
- U5 pad 19: GND -> AGND
- U5 pad 20: unconnected-(U5-TOCAP-Pad20) -> Net-(U5-TOCAP)
- U5 pad 21: Net-(U5-AVDD-Pad11) -> AVDD
- U5 pad 22: unconnected-(U5-1V2O-Pad22) -> Net-(U5-1V2O)
- U5 pad 28: unconnected-(U5-VDD-Pad28) -> +3V3
- U5 pad 3: GND -> AGND
- U5 pad 32: unconnected-(U5-~{SCS}-Pad32) -> /~{SCS}
- U5 pad 33: unconnected-(U5-SCLK-Pad33) -> /GPIO18
- U5 pad 34: unconnected-(U5-MISO-Pad34) -> /MISO
- U5 pad 35: unconnected-(U5-MOSI-Pad35) -> /GPIO19
- U5 pad 36: unconnected-(U5-~{INT}-Pad36) -> /~{INT}
- U5 pad 37: unconnected-(U5-~{RST}-Pad37) -> /~{RST}
- U5 pad 4: Net-(U5-AVDD-Pad11) -> AVDD
- U5 pad 43: unconnected-(U5-PMODE2-Pad43) -> /PMODE2
- U5 pad 44: unconnected-(U5-PMODE1-Pad44) -> /PMODE1
- U5 pad 45: unconnected-(U5-PMODE0-Pad45) -> /PMODE0
- U5 pad 48: GND -> AGND
- U5 pad 8: Net-(U5-AVDD-Pad11) -> AVDD
- U5 pad 9: GND -> AGND
- U6 pad 1: /CS -> /~{SCS}
- U6 pad 4: /MISO_MCU -> /GPIO20
Routing:
- net /GPIO20: track 0.00 -> 30.1 mm
- net /GPIO19: track 0.00 -> 29.4 mm, vias 0 -> 1
- net AVDD: track 0.00 -> 25.7 mm
- net /GPIO18: track 0.00 -> 24.1 mm, vias 0 -> 1
- net +3V3: track 1.22 -> 19.0 mm, vias 0 -> 1
- net AGND: track 0.00 -> 12.7 mm, vias 0 -> 1
- net /PMODE2: track 0.00 -> 7.91 mm, vias 0 -> 1
- net /PMODE1: track 0.00 -> 7.19 mm, vias 0 -> 1
- net /PMODE0: track 0.00 -> 6.56 mm, vias 0 -> 1
- net Net-(U5-TOCAP): track 0.00 -> 6.23 mm
- net /MISO: track 0.00 -> 5.37 mm
- net Net-(U5-LINKLED): track 0.00 -> 4.64 mm, vias 0 -> 1
- net Net-(U5-ACTLED): track 0.00 -> 4.06 mm, vias 0 -> 1
- net /~{SCS}: track 0.00 -> 3.88 mm
- net Net-(U5-1V2O): track 0.00 -> 3.46 mm
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- added copper zone on B.Cu, net AGND
- added copper zone on F.Cu, net AGND

Commit message: Need RJ45 alternative for W5500 not W5500s
Parts:
- added C13: 6.8nF, Capacitor_SMD:C_0402_1005Metric, F.Cu at (141.6, 112.1)
- added C14: 6.8nF, Capacitor_SMD:C_0402_1005Metric, F.Cu at (139.2, 112.1)
- added C15: 100nF, Capacitor_SMD:C_0402_1005Metric, F.Cu at (136.8, 112.1)
- added R10: 49.9, Resistor_SMD:R_0402_1005Metric, F.Cu at (138.0, 112.1)
- added R9: 49.9, Resistor_SMD:R_0402_1005Metric, F.Cu at (140.4, 112.1)
- added U1: RB1-125BAG1A, rb1-125bagia:WIZnet-RB1-125BAG1A-0, F.Cu at (136.4, 124.7)
- moved J3 58.1 mm to (190.9, 144.9)
- moved J8 45.6 mm to (162.9, 135.2)
- moved C18 0.41 mm to (135.6, 112.1)
- moved R18 0.14 mm to (134.5, 112.1)
- moved R17 0.07 mm to (133.3, 112.1)
Connections:
- C18 pad 1: GND -> AGND
- C18 pad 2: Net-(J8-TCT) -> Net-(U1-CT)
- J8 pad R4: Net-(J8-TCT) -> unconnected-(J8-TCT-PadR4)
- R18 pad 2: Net-(J8-TCT) -> Net-(U1-CT)
