File: W5500-hat.kicad_sch (KiCad schematic)
At the start: 28 parts, among them J1 Conn, J2 Conn, J3 RB1-125BAG1A, J4 Conn, J5 Conn, J8 RJ45_Amphenol_RJMG1BD3B8K1ANR, SW2 SW_Push, U5 W5500, U6 74AHC1G125, Y1 24MHz

Commit message: Tracks almost finished
Parts:
- added C10, C11, C5, C7: 100nF, Capacitor_SMD:C_0402_1005Metric, symbol Device:C_Small
- added C12, C6: 1uF, Capacitor_SMD:C_0603_1608Metric, symbol Device:C_Small
- added C4: 10uF, Capacitor_SMD:C_0603_1608Metric, symbol Device:C_Small
- added JP1, JP2, JP3: JMP, Jumper:SolderJumper-2_P1.3mm_Open_RoundedPad1.0x1.5mm, symbol Jumper:SolderJumper_2_Open
- added R4, R5, R6: 10K, Resistor_SMD:R_0402_1005Metric, symbol Device:R_Small
- added R7: 49.9, Resistor_SMD:R_0402_1005Metric, symbol Device:R_Small
- added R8: 17.4K, Resistor_SMD:R_0402_1005Metric, symbol Device:R_Small
- C9: value 1uF -> 100nF; footprint Capacitor_SMD:C_0603_1608Metric -> Capacitor_SMD:C_0402_1005Metric
Connections:
- net +1V2 is gone; now on net AVDD: C8.1, C9.1
- net CS is gone; now on net ~{SCS}: U6.1
- net MISO_MCU is gone; now on net GPIO20: U6.4
- net +3V3: now also U5.28 (VDD), C6.1, C7.1, R4.1, R5.1, R6.1, R7.1
- net AGND: now also C8.2, C9.2, U5.14 (AGND), U5.16 (AGND), U5.19 (AGND), U5.3 (AGND), U5.48 (AGND), U5.9 (AGND), C10.2, C11.2, C12.2, C4.2, C5.2, R8.2
- net AVDD: now also U5.11 (AVDD), U5.15 (AVDD), U5.17 (AVDD), U5.21 (AVDD), U5.4 (AVDD), U5.8 (AVDD), C10.1, C11.1, C12.1
- net GND: now also SW2.1, C6.2, C7.2, JP1.2 (B), JP2.2 (B), JP3.2 (B); no longer C8.2, C9.2, U5.14 (AGND), U5.16 (AGND), U5.19 (AGND), U5.3 (AGND), U5.48 (AGND), U5.9 (AGND)
- net GPIO18: now also U5.33 (SCLK)
- net GPIO19: now also U5.35 (MOSI)
- net MISO: now also U5.34 (MISO)
- net ~{RST}: now also SW2.2, U5.37 (~{RST}), R7.2
- net at U5.10 (EXRES1): now also R8.1
- net at U5.20 (TOCAP): now also C4.1
- net at U5.22 (1V2O): now also C5.1
- net ~{SCS}: now reaches U5.32 (~{SCS})
- net ~{INT}: now reaches U5.36 (~{INT})
- net PMODE2: now reaches U5.43 (PMODE2)
- net PMODE2: now also JP2.1 (A), R5.2
- net PMODE1: now reaches U5.44 (PMODE1)
- net PMODE1: now also JP1.1 (A), R4.2
- net PMODE0: now reaches U5.45 (PMODE0)
- net PMODE0: now also JP3.1 (A), R6.2
- no-connect marks 0 -> 9
Other:
- moved on the sheet: C1, C2, C3, C8, FB1, FB2, J1, J2, J4, J5, R1, R2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

Commit message: Need RJ45 alternative for W5500 not W5500s
Parts:
- added C13, C14: 6.8nF, Capacitor_SMD:C_0402_1005Metric, symbol Device:C_Small
- added C15: 100nF, Capacitor_SMD:C_0402_1005Metric, symbol Device:C_Small
- added R10, R9: 49.9, Resistor_SMD:R_0402_1005Metric, symbol Device:R_Small
- added U1: RB1-125BAG1A, rb1-125bagia:WIZnet-RB1-125BAG1A-0, symbol RJ45-MyLib:RB1-125BAG1A-MyLib
Connections:
- net +3V3: now also U1.L2 (LED_YELLOW-), U1.L4 (LED_GREEN-)
- net AGND: now also C18.1, C15.2
- net GND: now also U1.1 (SHIELD), U1.2 (SHIELD); no longer C18.1
- net GREEN_LED: now also U1.L3 (LED_GREEN+)
- net RXN: now also C13.1, R9.1
- net RXP: now also C14.1, R10.1
- net TXN: now also U1.R2 (TD-)
- net TXP: now also U1.R1 (TD+)
- net YELLOW_LED: now also U1.L1 (LED_YELLOW+)
- net at C18.2, R18.2: now also C15.1, R10.2, R9.2, U1.R3 (CT); no longer J8.R4 (TCT)
- new net: C14.2, U1.R7 (RD+)
- new net: C13.2, U1.R8 (RD-)
Other:
- moved on the sheet: C18, R16, R17, R18
